Commit message: did a lot of perception stack work

File: src/realsense_ros_gazebo/xacro/depthcam.xacro (robot description, xacro)
@@ -6,5 +6,5 @@
     <xacro:property name="d435_cam_depth_to_left_ir_offset" value="0.0"/>
     <xacro:property name="d435_cam_depth_to_right_ir_offset" value="-0.050"/>
-    <xacro:property name="d435_cam_depth_to_color_offset" value="0.015"/>
+    <xacro:property name="d435_cam_depth_to_color_offset" value="0.0"/>
     <xacro:property name="d435_cam_width" value="0.090"/>
     <xacro:property name="d435_cam_height" value="0.025"/>
@@ -177,8 +177,8 @@
       <sensor name="${sensor_name}_depth" type="depth">
         <camera name="${sensor_name}">
-          <horizontal_fov>${85.2*deg_to_rad}</horizontal_fov>
+          <horizontal_fov>${69.4*deg_to_rad}</horizontal_fov>
           <image>
-            <width>1280</width>
-            <height>720</height>
+            <width>640</width>
+            <height>480</height>
           </image>
           <clip>

File: src/turtlebot3/turtlebot3_description/urdf/turtlebot3_burger.urdf.xacro (robot description, xacro)
@@ -4,5 +4,5 @@
   <xacro:include filename="$(find turtlebot3_description)/urdf/turtlebot3_burger.gazebo.xacro"/>
   <xacro:include filename="$(find realsense_ros_gazebo)/xacro/depthcam.xacro"/>
-  <xacro:realsense_d435 sensor_name="d435" parent_link="base_link" rate="10">
+  <xacro:realsense_d435 sensor_name="/tb3_0/d435" parent_link="base_link" rate="10">
   <origin rpy="0 0 0 " xyz="-0.03 0 0.172"/>
   </xacro:realsense_d435>
@@ -11,4 +11,9 @@
     <parent link="base_footprint"/>
     <child link="base_link"/>
+    <origin xyz="0.0 0.0 0.010" rpy="0 0 0"/>
+  </joint>
+  <joint name="fill_joint" type="fixed">
+    <parent link="base_link"/>
+    <child link="fill_link"/>
     <origin xyz="0.0 0.0 0.010" rpy="0 0 0"/>
   </joint>
@@ -34,4 +39,13 @@
                izz="2.0064271e-03" />
     </inertial>
+  </link>
+    <link name="fill_link">
+    <visual>
+      <origin xyz="-0.032 0 0.05" rpy="0 0 0"/>
+      <geometry>
+        <cylinder length="0.15" radius="0.05"/>
+      </geometry>
+      <material name="light_black"/>
+    </visual>
   </link>
   <joint name="wheel_left_joint" type="continuous">
